File: ANALOG.kicad_sch (KiCad schematic)
At the start: 0 parts

Commit message: Rev e: nest INJ/LS DPAKs on frame, apply netlist, GND pours, route
Place Q1-Q7 + R1-R7 clear of AMPSEAL keepout; unify GND global net;
assign schematic nets to pads; add F/B GND zones and scripted frame
tracks/vias. Module copper remains Create Board gerber merge.
Changed lines of the file:
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@@
+		)
+	)
+	(wire
+		(pts
+			(xy 50.8 30.48) (xy 150 30.48)
+		)
+		(stroke
+			(width 0)
+			(type default)
+		)
+	)
+	(wire
+		(pts
+			(xy 50.8 40.64) (xy 150 40.64)
+		)
+		(stroke
+			(width 0)
+			(type default)
+		)
+	)
+	(wire
+		(pts
+			(xy 50.8 50.8) (xy 150 50.8)
+		)
+		(stroke
+			(width 0)
+			(type default)
+		)
+	)
+	(wire
+		(pts
+			(xy 50.8 60.959999999999994) (xy 150 60.959999999999994)
+		)
+		(stroke
+			(width 0)
+			(type default)
+		)
+	)
+	(wire
+		(pts
+			(xy 50.8 71.11999999999999) (xy 150 71.11999999999999)
+		)
+		(stroke
+			(width 0)
+			(type default)
+		)
+	)
+	(wire
+		(pts
+			(xy 50.8 81.27999999999999) (xy 150 81.27999999999999)
+		)
+		(stroke
+			(width 0)
+			(type default)
 		)
 	)
