File: INJ4.kicad_sch (KiCad schematic)
At the start: 20 parts, among them Q1 VND14NV04-E, Q2 VND14NV04-E, Q3 VND14NV04-E, Q4 VND14NV04-E

Commit message: Rev o: NCE4080K on Q1-Q7 and restore LS FETs
Swap every power FET from VND14NV04-E to NCE4080K (LCSC C191380,
TO-252-2L) on the existing DPAK land. Bring back Q5-Q7 and gate
R5-R7, and put AMPSEAL pins 8/9/10 back to fuel pump, idle, and boost.

F407VGT6 on mega-mcu100, injector TVS/flyback, Core EFI silk, GND
pours, and the drill origin stay. RDS(on) is rated at 10 V; the
3.3 V gate has no added driver.

Co-authored-by: Quintin <quintinbannink42@users.noreply.github.com>
Parts:
- Q1, Q2, Q3, Q4: value VND14NV04-E -> NCE4080K
Other:
- note added: "INJ4 Injectors rev O NCE4080K TO-252-2L (LCSC C191380) on microcore-fp:DPAK SMAJ33A (DO-214AC) + US1M UF flyback kept 2x12 ohm high-Z per channel (gate R1-R4 + ballast R8-R11) D1-D8 stay on B.Cu beside AMPSEAL J1"
- note removed: "INJ4 Injectors DPAK N-FET + SMAJ33A (DO-214AC) + US1M UF flyback 2x12 ohm high-Z per channel (gate R1-R4 + ballast R8-R11) rev K: D1-D8 on B.Cu beside AMPSEAL J1"
Changed lines of the file:
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@@
 	(title_block
 		(title "INJ4 Injectors")
-		(date "2026-09-13")
-		(rev "K")
+		(date "2026-09-22")
+		(rev "O")
 		(company "Core EFI")
+		(comment 1 "rev o: Q1-Q4 NCE4080K C191380; D1-D8 and R8-R11 kept")
 	)
 	(symbol
@@
 			)
 		)
-		(property "Value" "VND14NV04-E"
+		(property "Value" "NCE4080K"
 			(at 96.52 22.86 0)
 			(effects
@@
 			)
 		)
-		(property "Value" "VND14NV04-E"
+		(property "Value" "NCE4080K"
 			(at 96.52 53.339999999999996 0)
 			(effects
@@
 			)
 		)
-		(property "Value" "VND14NV04-E"
+		(property "Value" "NCE4080K"
 			(at 96.52 83.82 0)
 			(effects
@@
 			)
 		)
-		(property "Value" "VND14NV04-E"
+		(property "Value" "NCE4080K"
 			(at 96.52 114.3 0)
 			(effects
@@
 		)
 	)
-	(text "INJ4 Injectors\nDPAK N-FET + SMAJ33A (DO-214AC) + US1M UF flyback\n2x12 ohm high-Z per channel (gate R1-R4 + ballast R8-R11)\nrev K: D1-D8 on B.Cu beside AMPSEAL J1"
+	(text "INJ4 Injectors rev O\nNCE4080K TO-252-2L (LCSC C191380) on microcore-fp:DPAK\nSMAJ33A (DO-214AC) + US1M UF flyback kept\n2x12 ohm high-Z per channel (gate R1-R4 + ballast R8-R11)\nD1-D8 stay on B.Cu beside AMPSEAL J1"
 		(at 25.4 15.24 0)
 		(effects

Commit message: Rev p: AOD4184A on Q1-Q7, LS flyback+TVS, frame short fixes
Quintin chose AOD4184A (LCSC C99124) plus TVS for budget and reliability.
Q5-Q7 get the existing US1M flyback and SMAJ33A. Injector/VR frame shorts
on the board copper are cleared; Hellen module pad-G noise stays documented.

Co-authored-by: Quintin <quintinbannink42@users.noreply.github.com>
Parts:
- Q1, Q2, Q3, Q4: value NCE4080K -> AOD4184A
Other:
- note added: "INJ4 Injectors rev P AOD4184A TO-252 (LCSC C99124) on microcore-fp:DPAK SMAJ33A (DO-214AC) + US1M UF flyback kept 2x12 ohm high-Z per channel (gate R1-R4 + ballast R8-R11) D1-D8 stay on B.Cu beside AMPSEAL J1 RDS(on) max 9.5 mohm at 4.5 V; Vth max 2.6 V; MCU gate is 3.3 V"
- note removed: "INJ4 Injectors rev O NCE4080K TO-252-2L (LCSC C191380) on microcore-fp:DPAK SMAJ33A (DO-214AC) + US1M UF flyback kept 2x12 ohm high-Z per channel (gate R1-R4 + ballast R8-R11) D1-D8 stay on B.Cu beside AMPSEAL J1"
Changed lines of the file:
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@@
 	(title_block
 		(title "INJ4 Injectors")
-		(date "2026-09-22")
-		(rev "O")
+		(date "2026-09-24")
+		(rev "P")
 		(company "Core EFI")
-		(comment 1 "rev o: Q1-Q4 NCE4080K C191380; D1-D8 and R8-R11 kept")
+		(comment 1 "rev p: Q1-Q4 AOD4184A C99124; D1-D8 and R8-R11 kept")
 	)
 	(symbol
@@
 			)
 		)
-		(property "Value" "NCE4080K"
+		(property "Value" "AOD4184A"
 			(at 96.52 22.86 0)
 			(effects
@@
 			)
 		)
-		(property "Value" "NCE4080K"
+		(property "Value" "AOD4184A"
 			(at 96.52 53.339999999999996 0)
 			(effects
@@
 			)
 		)
-		(property "Value" "NCE4080K"
+		(property "Value" "AOD4184A"
 			(at 96.52 83.82 0)
 			(effects
@@
 			)
 		)
-		(property "Value" "NCE4080K"
+		(property "Value" "AOD4184A"
 			(at 96.52 114.3 0)
 			(effects
@@
 		)
 	)
-	(text "INJ4 Injectors rev O\nNCE4080K TO-252-2L (LCSC C191380) on microcore-fp:DPAK\nSMAJ33A (DO-214AC) + US1M UF flyback kept\n2x12 ohm high-Z per channel (gate R1-R4 + ballast R8-R11)\nD1-D8 stay on B.Cu beside AMPSEAL J1"
+	(text "INJ4 Injectors rev P\nAOD4184A TO-252 (LCSC C99124) on microcore-fp:DPAK\nSMAJ33A (DO-214AC) + US1M UF flyback kept\n2x12 ohm high-Z per channel (gate R1-R4 + ballast R8-R11)\nD1-D8 stay on B.Cu beside AMPSEAL J1\nRDS(on) max 9.5 mohm at 4.5 V; Vth max 2.6 V; MCU gate is 3.3 V"
 		(at 25.4 15.24 0)
 		(effects

Commit message: Rev p: keep Q1-Q7 as NCE4080K; LS US1M+SMAJ33A stays
Budget and reliability first. No FET or BOM upgrade and no DPAK land change. Low-side clamps stay the injector US1M and SMAJ33A already in the BOM.

Co-authored-by: Quintin <quintinbannink42@users.noreply.github.com>
Parts:
- Q1, Q2, Q3, Q4: value AOD4184A -> NCE4080K
Other:
- note added: "INJ4 Injectors rev P NCE4080K TO-252 (LCSC C191380) on microcore-fp:DPAK SMAJ33A (DO-214AC) + US1M UF flyback kept 2x12 ohm high-Z per channel (gate R1-R4 + ballast R8-R11) D1-D8 stay on B.Cu beside AMPSEAL J1 RDS(on) at 10 V only (<7 mohm); Vth max 2.5 V; MCU gate is 3.3 V"
- note removed: "INJ4 Injectors rev P AOD4184A TO-252 (LCSC C99124) on microcore-fp:DPAK SMAJ33A (DO-214AC) + US1M UF flyback kept 2x12 ohm high-Z per channel (gate R1-R4 + ballast R8-R11) D1-D8 stay on B.Cu beside AMPSEAL J1 RDS(on) max 9.5 mohm at 4.5 V; Vth max 2.6 V; MCU gate is 3.3 V"
Changed lines of the file:
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@@
 		(rev "P")
 		(company "Core EFI")
-		(comment 1 "rev p: Q1-Q4 AOD4184A C99124; D1-D8 and R8-R11 kept")
+		(comment 1 "rev p: Q1-Q4 stay NCE4080K C191380; D1-D8 and R8-R11 kept")
 	)
 	(symbol
@@
 			)
 		)
-		(property "Value" "AOD4184A"
+		(property "Value" "NCE4080K"
 			(at 96.52 22.86 0)
 			(effects
@@
 			)
 		)
-		(property "Value" "AOD4184A"
+		(property "Value" "NCE4080K"
 			(at 96.52 53.339999999999996 0)
 			(effects
@@
 			)
 		)
-		(property "Value" "AOD4184A"
+		(property "Value" "NCE4080K"
 			(at 96.52 83.82 0)
 			(effects
@@
 			)
 		)
-		(property "Value" "AOD4184A"
+		(property "Value" "NCE4080K"
 			(at 96.52 114.3 0)
 			(effects
@@
 		)
 	)
-	(text "INJ4 Injectors rev P\nAOD4184A TO-252 (LCSC C99124) on microcore-fp:DPAK\nSMAJ33A (DO-214AC) + US1M UF flyback kept\n2x12 ohm high-Z per channel (gate R1-R4 + ballast R8-R11)\nD1-D8 stay on B.Cu beside AMPSEAL J1\nRDS(on) max 9.5 mohm at 4.5 V; Vth max 2.6 V; MCU gate is 3.3 V"
+	(text "INJ4 Injectors rev P\nNCE4080K TO-252 (LCSC C191380) on microcore-fp:DPAK\nSMAJ33A (DO-214AC) + US1M UF flyback kept\n2x12 ohm high-Z per channel (gate R1-R4 + ballast R8-R11)\nD1-D8 stay on B.Cu beside AMPSEAL J1\nRDS(on) at 10 V only (<7 mohm); Vth max 2.5 V; MCU gate is 3.3 V"
 		(at 25.4 15.24 0)
 		(effects
