File: LS3.kicad_sch (KiCad schematic)
At the start: 12 parts, among them Q5 AOD4184A, Q6 AOD4184A, Q7 AOD4184A

Commit message: Rev q: NCE4080K (C191380) plus SLM27524 gate drivers on V12_RAW
Restore Q1-Q7 to NCE4080K and insert four SLM27524CA-DG drivers so the
STM32 GPIO no longer drives the FET gates. Seven channels are used; the
spare input is tied to GND. LS clamps and the rev p short fixes stay.

Co-authored-by: Quintin <quintinbannink42@users.noreply.github.com>
Parts:
- added C5, C7: 100n, microcore-fp:C0603, symbol microcore:C
- added C6, C8: 1u, microcore-fp:C0603, symbol microcore:C
- added U3, U4: SLM27524CA-DG, microcore-fp:SOIC-8, symbol microcore:SLM27524
- Q5, Q6, Q7: value AOD4184A -> NCE4080K
Connections:
- net GND: now also C5.1, C6.1, C7.1, C8.1, U3.3 (GND), U4.2 (INA), U4.3 (GND)
- net IN1: now also U3.4 (INB); no longer R5.2
- net IN2: now also U3.2 (INA); no longer R6.2
- net IN3: now also U4.4 (INB); no longer R7.2
- net OUT2: now also C5.2, C6.2, C7.2, C8.2, U3.1 (ENA), U3.6 (VDD), U3.8 (ENB), U4.1 (ENA), U4.6 (VDD), U4.8 (ENB)
- new net: R7.2, U4.5 (OUTB)
- new net: R5.2, U3.5 (OUTB)
- new net: R6.2, U3.7 (OUTA)
- no-connect marks 0 -> 1
Other:
- note added: "LS3 Low-side rev Q Q5-Q7 NCE4080K TO-252 (LCSC C191380) on microcore-fp:DPAK Gate path: MCU GPIO to SLM27524CA-DG (VDD = V12_RAW) to R5-R7 12 ohm US1M flyback (C112545) + SMAJ33A (C143131); no series ballast U4 channel A input tied to GND; OUTA unused"
- note removed: "LS3 Low-side rev P Q5-Q7 AOD4184A TO-252 (LCSC C99124) on microcore-fp:DPAK 12 ohm gate; US1M flyback (C112545) + SMAJ33A (C143131); no series ballast Discrete MOSFET, not a protected smart FET. No gate driver. No premium clamps. RDS(on) max 9.5 mohm at Vgs=4.5 V (not specified at 3.3 V). Vth max 2.6 V. MCU gate is 3.3 V, so the FET turns on but Rds at 3.3 V is not guaranteed."
